File: ISA8888_KiCAD/ISA8888.kicad_pcb (KiCad board)
At the start: 2 copper layers, 1 part, among them U2 AT24CS02-SSHM

Commit message: ISA8888 rev00
Parts:
- added C1: 100uF, Capacitor_THT:CP_Radial_D5.0mm_P2.50mm, F.Cu at (82.2, 77.2)
- added C10: 100nF, Capacitor_SMD:C_1808_4520Metric_Pad1.72x2.30mm_HandSolder, F.Cu at (98.1, 79.8)
- added C11: 100nF, Capacitor_SMD:C_1808_4520Metric_Pad1.72x2.30mm_HandSolder, F.Cu at (98.1, 83.6)
- added C12: 100nF, Capacitor_SMD:C_1808_4520Metric_Pad1.72x2.30mm_HandSolder, F.Cu at (98.1, 87.5)
- added C13: 100nF, Capacitor_SMD:C_1808_4520Metric_Pad1.72x2.30mm_HandSolder, F.Cu at (98.1, 91.3)
- added C14: 100nF, Capacitor_SMD:C_1808_4520Metric_Pad1.72x2.30mm_HandSolder, F.Cu at (98.1, 95.2)
- added C15: 47uF, Capacitor_THT:CP_Radial_D5.0mm_P2.50mm, F.Cu at (82.2, 83.8)
- added C16: 100nF, Capacitor_SMD:C_1808_4520Metric_Pad1.72x2.30mm_HandSolder, F.Cu at (98.1, 99.0)
- added C17: 100nF, Capacitor_SMD:C_1808_4520Metric_Pad1.72x2.30mm_HandSolder, F.Cu at (105.7, 75.9)
- added C18: 47uF, Capacitor_THT:CP_Radial_D5.0mm_P2.50mm, F.Cu at (82.2, 90.3)
- added C19: 100nF, Capacitor_SMD:C_1808_4520Metric_Pad1.72x2.30mm_HandSolder, F.Cu at (105.7, 79.8)
- added C2: 100nF, Capacitor_SMD:C_1808_4520Metric_Pad1.72x2.30mm_HandSolder, F.Cu at (90.5, 75.9)
- added C20: 100nF, Capacitor_SMD:C_1808_4520Metric_Pad1.72x2.30mm_HandSolder, F.Cu at (105.7, 83.6)
- added C21: 100nF, Capacitor_SMD:C_1808_4520Metric_Pad1.72x2.30mm_HandSolder, F.Cu at (105.7, 87.5)
- added C22: 100nF, Capacitor_SMD:C_1808_4520Metric_Pad1.72x2.30mm_HandSolder, F.Cu at (105.7, 91.3)
- added C23: 100nF, Capacitor_SMD:C_1808_4520Metric_Pad1.72x2.30mm_HandSolder, F.Cu at (105.7, 95.2)
- added C24: 100nF, Capacitor_SMD:C_1808_4520Metric_Pad1.72x2.30mm_HandSolder, F.Cu at (105.7, 99.0)
- added C25: 100nF, Capacitor_SMD:C_1808_4520Metric_Pad1.72x2.30mm_HandSolder, F.Cu at (113.3, 75.9)
- added C26: 100nF, Capacitor_SMD:C_1808_4520Metric_Pad1.72x2.30mm_HandSolder, F.Cu at (113.3, 79.8)
- added C27: 100nF, Capacitor_SMD:C_1808_4520Metric_Pad1.72x2.30mm_HandSolder, F.Cu at (113.3, 83.6)
- added C28: 100nF, Capacitor_SMD:C_1808_4520Metric_Pad1.72x2.30mm_HandSolder, F.Cu at (113.3, 87.5)
- added C29: 100nF, Capacitor_SMD:C_1808_4520Metric_Pad1.72x2.30mm_HandSolder, F.Cu at (113.3, 91.3)
- added C3: 100nF, Capacitor_SMD:C_1808_4520Metric_Pad1.72x2.30mm_HandSolder, F.Cu at (90.5, 79.8)
- added C30: 100uF, Capacitor_THT:CP_Radial_D5.0mm_P2.50mm, F.Cu at (82.2, 96.9)
- added C31: 100nF, Capacitor_SMD:C_1808_4520Metric_Pad1.72x2.30mm_HandSolder, F.Cu at (113.3, 95.2)
- added C32: 100nF, Capacitor_SMD:C_1808_4520Metric_Pad1.72x2.30mm_HandSolder, F.Cu at (113.3, 99.0)
- added C33: 100uF, Capacitor_THT:CP_Radial_D5.0mm_P2.50mm, F.Cu at (82.2, 103.5)
- added C4: 100nF, Capacitor_SMD:C_1808_4520Metric_Pad1.72x2.30mm_HandSolder, F.Cu at (90.5, 83.6)
- added C5: 100nF, Capacitor_SMD:C_1808_4520Metric_Pad1.72x2.30mm_HandSolder, F.Cu at (90.5, 87.5)
- added C6: 100nF, Capacitor_SMD:C_1808_4520Metric_Pad1.72x2.30mm_HandSolder, F.Cu at (90.5, 91.3)
- added C7: 100nF, Capacitor_SMD:C_1808_4520Metric_Pad1.72x2.30mm_HandSolder, F.Cu at (90.5, 95.2)
- added C8: 100nF, Capacitor_SMD:C_1808_4520Metric_Pad1.72x2.30mm_HandSolder, F.Cu at (90.5, 99.0)
- added C9: 100nF, Capacitor_SMD:C_1808_4520Metric_Pad1.72x2.30mm_HandSolder, F.Cu at (98.1, 75.9)
- added J1: Bus_PCI_32bit_Universal, Connector_PCBEdge:BUS_PCI, F.Cu at (119.8, 140.8)
- added J2: Bus_ISA_16bit, ISA8888:CONN_EBC49_SUL, F.Cu at (219.3, 57.4)
- added J3: Conn_02x03, Connector_PinHeader_2.00mm:PinHeader_2x03_P2.00mm_Vertical, F.Cu at (99.5, 112.3)
- added J4: Conn_02x02, Connector_PinHeader_2.00mm:PinHeader_2x02_P2.00mm_Vertical, F.Cu at (142.5, 43.0)
- added R10: R330, Resistor_THT:R_Axial_DIN0204_L3.6mm_D1.6mm_P5.08mm_Horizontal, F.Cu at (158.0, 121.7)
- added R11: R330, Resistor_THT:R_Axial_DIN0204_L3.6mm_D1.6mm_P5.08mm_Horizontal, F.Cu at (161.5, 121.8)
- added R12: R330, Resistor_THT:R_Axial_DIN0204_L3.6mm_D1.6mm_P5.08mm_Horizontal, F.Cu at (172.0, 121.8)
- added R13: R4.7K, Resistor_THT:R_Axial_DIN0204_L3.6mm_D1.6mm_P5.08mm_Horizontal, F.Cu at (128.5, 110.3)
- added R14: R4.7K, Resistor_THT:R_Axial_DIN0204_L3.6mm_D1.6mm_P5.08mm_Horizontal, F.Cu at (128.5, 112.8)
- added R15: R50K, Resistor_THT:R_Axial_DIN0204_L3.6mm_D1.6mm_P5.08mm_Horizontal, F.Cu at (161.0, 82.9)
- added R16: R50K, Resistor_THT:R_Axial_DIN0204_L3.6mm_D1.6mm_P5.08mm_Horizontal, F.Cu at (154.0, 82.8)
- added R17: R50K, Resistor_THT:R_Axial_DIN0204_L3.6mm_D1.6mm_P5.08mm_Horizontal, F.Cu at (157.5, 82.8)
- added R3: R4.7K, Resistor_THT:R_Axial_DIN0204_L3.6mm_D1.6mm_P5.08mm_Horizontal, F.Cu at (107.5, 110.3)
- added R4: R4.7K, Resistor_THT:R_Axial_DIN0204_L3.6mm_D1.6mm_P5.08mm_Horizontal, F.Cu at (107.5, 114.3)
- added R5: R4.7K, Resistor_THT:R_Axial_DIN0204_L3.6mm_D1.6mm_P5.08mm_Horizontal, F.Cu at (107.5, 118.3)
- added R6: R4.7K, Resistor_THT:R_Axial_DIN0204_L3.6mm_D1.6mm_P5.08mm_Horizontal, F.Cu at (168.5, 121.8)
- added R7: R1K, Resistor_THT:R_Axial_DIN0204_L3.6mm_D1.6mm_P5.08mm_Horizontal, F.Cu at (165.0, 121.7)
- added R8: R1K, Resistor_THT:R_Axial_DIN0204_L3.6mm_D1.6mm_P5.08mm_Horizontal, F.Cu at (154.5, 121.7)
- added R9: R330, Resistor_THT:R_Axial_DIN0204_L3.6mm_D1.6mm_P5.08mm_Horizontal, F.Cu at (175.5, 121.7)
- added RN1: R_Net_10_10k, Resistor_THT:R_Array_SIP11, F.Cu at (126.0, 124.3)
- added RN2: R_Net_10_4k7, Resistor_THT:R_Array_SIP11, F.Cu at (189.5, 113.8)
- added RN3: R_Net_10_10k, Resistor_THT:R_Array_SIP11, F.Cu at (184.0, 88.4)
- added RN4: R_Net_10_10k, Resistor_THT:R_Array_SIP11, F.Cu at (178.5, 101.1)
- added U1: ~, Package_QFP:PQFP-160_28x28mm_P0.65mm, F.Cu at (153.5, 102.8)
- added Y1: CFPS-72, Oscillator:Oscillator_SMD_IQD_IQXO70-4Pin_7.5x5.0mm, F.Cu at (134.5, 44.0)
- moved U2 39.8 mm to (121.0, 110.3)

Commit message: Temp
Parts:
- moved C33 142.4 mm to (211.5, 43.8), turned to 90 degrees
- moved C6 133.3 mm to (217.2, 50.0), turned to 90 degrees
- moved C32 111.3 mm to (213.2, 50.0), turned to 90 degrees
- moved C13 109.0 mm to (199.0, 50.0), turned to 90 degrees
- moved C19 107.7 mm to (209.2, 50.0), turned to 90 degrees
- moved C17 101.6 mm to (204.0, 50.0), turned to 90 degrees
- moved C3 98.5 mm to (186.5, 102.0)
- moved C7 97.3 mm to (186.5, 111.0)
- moved C1 88.5 mm to (155.0, 127.5), turned to 90 degrees
- moved C11 80.2 mm to (178.0, 76.0), turned to 90 degrees
- moved C2 73.5 mm to (150.0, 119.0), turned to -90 degrees
- moved C21 69.2 mm to (174.0, 76.0), turned to 90 degrees
- moved C4 60.4 mm to (140.8, 50.0), turned to 90 degrees
- moved C12 60.3 mm to (144.2, 126.3), turned to 90 degrees
- moved C30 56.8 mm to (130.0, 127.5), turned to 90 degrees
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Other:
- board outline added: 154.8 x 106.2 mm
