File: ISA8888_KiCAD/ISA8888_RoutingTest.kicad_pcb (KiCad board)
At the start: 2 copper layers, 154.8 x 106.2 mm, 65 parts, among them J1 Bus_PCI_32bit_Universal, J2 Bus_ISA_16bit, J3 AEN/BALE/TC J3, J4 Crystal J4, J5 PCI Jumpers, J6 PPDGNT# Motherboard Redirect, J7 PPDREQ# Motherboard Redirect, U2 SMROM-AT24CS02, U3 -5v MAX660, Y1 CFPS-72

Commit message: Routing Test + MAX660
Parts:
- moved J3 34.8 mm to (119.7, 73.3), turned to -90 degrees
- moved C33 0.97 mm to (212.3, 43.2), turned to 180 degrees
- moved R7 0.79 mm to (180.5, 117.0)
- moved R9 0.79 mm to (191.0, 117.0)
- moved R11 0.75 mm to (177.0, 117.0)
- moved R12 0.75 mm to (187.5, 117.0)
- moved R6 0.75 mm to (184.0, 117.0)
- moved R10 0.74 mm to (173.5, 117.0)
- moved R8 0.74 mm to (170.0, 117.0)
- moved C17 0.15 mm to (204.2, 50.0)
- moved C19 0.10 mm to (209.2, 50.0)
Routing:
- net GND: track 0.00 -> 795.8 mm, vias 0 -> 18
- net +5V: track 0.00 -> 639.8 mm, vias 0 -> 8
- net +3.3V: track 0.00 -> 237.9 mm, vias 0 -> 9
- net -12V: track 0.00 -> 219.5 mm, vias 0 -> 2
- net +12V: track 0.00 -> 209.8 mm, vias 0 -> 3
- net -5V: track 0.00 -> 65.9 mm
- net Net-(J3-Pin_6): track 0.00 -> 38.4 mm
- net Net-(J3-Pin_4): track 0.00 -> 34.2 mm
- net Net-(J3-Pin_2): track 0.00 -> 30.2 mm
- net DRQ0: track 0.00 -> 27.1 mm, vias 0 -> 1
- net DRQ1: track 0.00 -> 25.7 mm, vias 0 -> 1
- net DRQ2: track 0.00 -> 23.9 mm, vias 0 -> 1
- net DRQ3: track 0.00 -> 22.2 mm, vias 0 -> 1
- net DRQ5: track 0.00 -> 20.5 mm, vias 0 -> 1
- net NOWS#: track 0.00 -> 20.3 mm
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