File: ISA8888_KiCAD/ISA8888_Test3.kicad_pcb (KiCad board)
At the start: 2 copper layers, 154.8 x 106.2 mm, 70 parts, among them J1 Bus_PCI_32bit_Universal, J2 Bus_ISA_16bit, J3 BALE/AEN/TC J3, J4 Crystal J4, J5 PCI Jumpers, J6 PPDGNT# Motherboard Redirect, J7 PPDREQ# Motherboard Redirect, U2 SMROM-AT24CS02, U4 LM7905_TO220, Y1 CFPS-72

Commit message: Fix negative cap orientations in SCH
Parts:
- moved C1 8.04 mm to (223.6, 96.9)
Routing:
- net GND: track 46.5 -> 798.0 mm, vias 0 -> 9
- net +5V: track 25.4 -> 490.0 mm, vias 0 -> 5
- net +3.3V: track 15.7 -> 357.9 mm, vias 0 -> 6
- net -12V: track 0.00 -> 333.4 mm, vias 0 -> 2
- net +12V: track 0.00 -> 267.9 mm, vias 0 -> 2
- net SA12: track 0.00 -> 135.3 mm, vias 0 -> 2
- net MEMCS16#: track 0.00 -> 126.5 mm, vias 0 -> 3
- net -5V: track 0.00 -> 124.4 mm
- net RSTDRV: track 0.00 -> 122.5 mm, vias 0 -> 2
- net SA8: track 0.00 -> 118.9 mm, vias 0 -> 2
- net SA9: track 0.00 -> 118.9 mm, vias 0 -> 2
- net IOW#: track 0.00 -> 113.3 mm, vias 0 -> 3
- net SA6: track 0.00 -> 113.0 mm, vias 0 -> 3
- net SA7: track 0.00 -> 110.2 mm, vias 0 -> 2
- net SA10: track 0.00 -> 108.6 mm, vias 0 -> 1
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