File: ISA8888_KiCAD/PowerConfig.kicad_sch (KiCad schematic)
At the start: 0 parts

Commit message: Fixup Power/Config Sheet and update PCB with info from P/C sheet
Parts:
- added C1, C30, C33: 100uF, Capacitor_THT:CP_Radial_D5.0mm_P2.50mm, symbol Device:C_US
- added C10, C11, C12, C13, C14, C16, C17, C19, C2, C20, C21, C22, C23, C24, C25, C26, C27, C28, C29, C3, C31, C32, C4, C5, C6, C7, C8, C9: 100nF, Capacitor_SMD:C_1808_4520Metric_Pad1.72x2.30mm_HandSolder, symbol Device:C_US
- added C15, C18: 47uF, Capacitor_THT:CP_Radial_D5.0mm_P2.50mm, symbol Device:C_US
- added C34, C35: 150uF, Capacitor_THT:CP_Radial_D5.0mm_P2.50mm, symbol Device:C_US
- added C36, C37: 33uF, Capacitor_THT:CP_Radial_D5.0mm_P2.50mm, symbol Device:C_US
- added D1: -5V, LED_THT:LED_D5.0mm, symbol Device:LED
- added J3: AEN/BALE/TC J3, Connector_PinHeader_2.00mm:PinHeader_2x03_P2.00mm_Vertical, symbol Connector_Generic:Conn_02x03_Odd_Even
- added J4: Crystal J4, Connector_PinHeader_2.00mm:PinHeader_2x02_P2.00mm_Vertical, symbol Connector_Generic:Conn_02x02_Top_Bottom
- added J5: PCI Jumpers, Connector_PinHeader_2.00mm:PinHeader_2x04_P2.00mm_Vertical, symbol Connector_Generic:Conn_02x04_Top_Bottom
- added J6: PPDGNT# Motherboard Redirect, Connector_PinHeader_2.00mm:PinHeader_1x01_P2.00mm_Vertical, symbol Connector:Conn_01x01_Pin
- added J7: PPDREQ# Motherboard Redirect, Connector_PinHeader_2.00mm:PinHeader_1x01_P2.00mm_Vertical, symbol Connector:Conn_01x01_Pin
- added R1: 330, Resistor_THT:R_Axial_DIN0207_L6.3mm_D2.5mm_P7.62mm_Horizontal, symbol Device:R
- added R10, R11, R12, R9: R330, Resistor_THT:R_Axial_DIN0204_L3.6mm_D1.6mm_P5.08mm_Horizontal, symbol Device:R
- added R13, R14, R3, R4, R5, R6: R4.7K, Resistor_THT:R_Axial_DIN0204_L3.6mm_D1.6mm_P5.08mm_Horizontal, symbol Device:R
- added R15, R16, R17: R50K, Resistor_THT:R_Axial_DIN0204_L3.6mm_D1.6mm_P5.08mm_Horizontal, symbol Device:R
- added R7, R8: R1K, Resistor_THT:R_Axial_DIN0204_L3.6mm_D1.6mm_P5.08mm_Horizontal, symbol Device:R
- added RN1, RN3, RN4: R_Net_10_10k, Resistor_THT:R_Array_SIP11, symbol Device:R_Network10
- added RN2: R_Net_10_4k7, Resistor_THT:R_Array_SIP11, symbol Device:R_Network10
- added U2: SMROM-AT24CS02, Package_SO:SOIC-8_3.9x4.9mm_P1.27mm, symbol Memory_EEPROM:AT24CS02-SSHM
- added U3: ~, Package_SO:SOIC-8_3.9x4.9mm_P1.27mm, symbol ISA8888:MAX660CSAT
- added U4: LM7905_TO220, Package_TO_SOT_THT:TO-220-3_Vertical, symbol Regulator_Linear:LM7905_TO220
- added Y1: CFPS-72, Oscillator:Oscillator_SMD_IQD_IQXO70-4Pin_7.5x5.0mm, symbol Oscillator:CFPS-72
Connections:
- new net: D1.1 (K), R1.2
- new net: J4.3 (Pin_3), J4.4 (Pin_4), Y1.1 (EN)
- new net: J3.2 (Pin_2), R3.1
- new net: J3.4 (Pin_4), R4.1
- new net: J3.6 (Pin_6), R5.1
- new net: C34.1, U3.2 (CAP+)
- new net: C34.2, U3.4 (CAP-)
- new net +12V: C13.1, C14.1, C15.1
- new net +3.3V: C20.1, C21.1, C22.1, C23.1, C24.1, C25.1, C26.1, C27.1, C28.1, C29.1, C30.1, C31.1, R15.2, R16.2, R17.2, U2.8 (VCC)
- new net +5V: C1.1, C10.1, C11.1, C12.1, C2.1, C3.1, C4.1, C5.1, C6.1, C7.1, C8.1, C9.1, J4.1 (Pin_1), R10.2, R11.2, R12.2, R6.2, R7.2, R8.2, R9.2, RN2.1 (common), RN3.1 (common), RN4.1 (common), U3.8 (V+), Y1.4 (+Vs)
- new net -12V: C16.1, C17.1, C18.1, C37.2, U4.2 (VI)
- new net -5V: C19.1, C32.1, C33.1, C35.2, C36.2, R1.1, U3.5 (OUT), U4.3 (VO)
- new net AEN: J3.1 (Pin_1)
- new net BALE: J3.3 (Pin_3)
- new net DRQ0: RN1.8 (R7)
- new net DRQ1: RN1.7 (R6)
- new net DRQ2: RN1.6 (R5)
- new net DRQ3: RN1.5 (R4)
- new net DRQ5: RN1.4 (R3)
- new net DRQ6: RN1.3 (R2)
- new net DRQ7: RN1.2 (R1)
- new net GND: C1.2, C10.2, C11.2, C12.2, C13.2, C14.2, C15.2, C16.2, C17.2, C18.2, C19.2, C2.2, C20.2, C21.2, C22.2, C23.2, C24.2, C25.2, C26.2, C27.2, C28.2, C29.2, C3.2, C30.2, C31.2, C32.2, C33.2, C35.1, C36.1, C37.1, C4.2, C5.2, C6.2, C7.2, C8.2, C9.2, D1.2 (A), J4.2 (Pin_2), R3.2, R4.2, R5.2, RN1.1 (common), U2.1 (A0), U2.2 (A1), U2.3 (A2), U2.4 (GND), U2.7 (WP), U3.3 (GND), U3.6 (LV), U4.1 (GND), Y1.2 (GND)
- new net IGNT#: J5.1 (Pin_1), J5.3 (Pin_3), J5.7 (Pin_7), R16.1
- new net IOCHCK#: R7.1
- new net IOCHRDY: R6.1
- new net IOCS16#: R10.1
- new net IOR#: RN2.2 (R1)
- new net IOW#: RN2.3 (R2)
- new net IREQ#: J5.2 (Pin_2), J5.4 (Pin_4), J5.8 (Pin_8)
- new net MASTER#: R12.1
- new net MB_PPDGNT#: J5.5 (Pin_5), J6.1 (Pin_1), R15.1
- new net MB_PPDREQ#: J5.6 (Pin_6), J7.1 (Pin_1)
- new net MEMCS16#: R11.1
- new net MEMR#: RN2.6 (R5)
- new net MEMW#: RN2.7 (R6)
- new net NOWS#: R9.1
- new net OSC: Y1.3 (Output)
- new net REFRESH#: R8.1
- new net SCL: R14.1, R14.2, U2.6 (SCL)
- new net SD0: RN3.9 (R8)
- new net SD1: RN3.8 (R7)
- new net SD10: RN4.4 (R3)
- new net SD11: RN4.5 (R4)
- new net SD12: RN4.6 (R5)
- new net SD13: RN4.7 (R6)
- new net SD14: RN4.8 (R7)
- new net SD15: RN4.9 (R8)
- new net SD2: RN3.7 (R6)
- new net SD3: RN3.6 (R5)
- new net SD4: RN3.5 (R4)
- new net SD5: RN3.4 (R3)
- new net SD6: RN3.3 (R2)
- new net SD7: RN3.2 (R1)
- new net SD8: RN4.2 (R1)
- new net SD9: RN4.3 (R2)
- new net SDA: R13.1, R13.2, U2.5 (SDA)
- new net SERIRQ: R17.1
- new net SMEMR#: RN2.4 (R3)
- new net SMEMW#: RN2.5 (R4)
- new net TC: J3.5 (Pin_5)
- no-connect marks 0 -> 13

Commit message: Fix negative cap orientations in SCH
Connections:
- net -12V: now also C16.2, C17.2, C18.2; no longer C16.1, C17.1, C18.1
- net -5V: now also C19.2, C32.2, C33.2; no longer C19.1, C32.1, C33.1
- net AEN: now also J3.3 (Pin_3); no longer J3.1 (Pin_1)
- net BALE: now also J3.1 (Pin_1); no longer J3.3 (Pin_3)
- net GND: now also C16.1, C17.1, C18.1, C19.1, C32.1, C33.1; no longer C16.2, C17.2, C18.2, C19.2, C32.2, C33.2
Other:
- moved on the sheet: C16, C17, C18, C19, C32, C33
Changed lines of the file:
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@@
 		)
 	)
-	(text_box "J3 - Jumper Functions\n\n1-2 OFF - Enable Chip test with PCIRST#=0\n	 ON - IT8888 Normal Function\n\n3-4 OFF - Fast DEVSEL# decode for F-Seg\n	 ON - No F-Seg decoding\n\n5-6 OFF - Enable SM Boot-ROM\n	 ON - Disable SM Boot-ROM"
+	(text_box "J3 - Jumper Functions\n\nBALE:\n1-2 OFF - Fast DEVSEL# decode for F-Seg\n	 ON - No F-Seg decoding\nAEN:\n3-4 OFF - Enable Chip test with PCIRST#=0\n	 ON - IT8888 Normal Function\nTC:\n5-6 OFF - Enable SM Boot-ROM\n	 ON - Disable SM Boot-ROM"
 		(exclude_from_sim no)
 		(at 304.8 134.62 0)
@@
 	)
 	(junction
-		(at 48.26 134.62)
+		(at 148.59 177.8)
 		(diameter 0)
 		(color 0 0 0 0)
 	)
 	(junction
-		(at 16.51 177.8)
+		(at 48.26 134.62)
 		(diameter 0)
 		(color 0 0 0 0)
 	)
 	(junction
-		(at 67.31 170.18)
+		(at 16.51 177.8)
 		(diameter 0)
 		(color 0 0 0 0)
 	)
 	(junction
-		(at 194.31 170.18)
+		(at 67.31 170.18)
 		(diameter 0)
 		(color 0 0 0 0)
@@
 	)
 	(junction
-		(at 26.67 189.23)
+		(at 158.75 177.8)
 		(diameter 0)
 		(color 0 0 0 0)
 	)
 	(junction
-		(at 26.67 170.18)
+		(at 26.67 189.23)
 		(diameter 0)
 		(color 0 0 0 0)
 	)
 	(junction
-		(at 158.75 177.8)
+		(at 26.67 170.18)
 		(diameter 0)
 		(color 0 0 0 0)
@@
 	)
 	(junction
-		(at 158.75 170.18)
-		(diameter 0)
-		(color 0 0 0 0)
-	)
-	(junction
 		(at 16.51 189.23)
 		(diameter 0)
@@
 	)
 	(junction
-		(at 184.15 170.18)
+		(at 26.67 196.85)
 		(diameter 0)
 		(color 0 0 0 0)
 	)
 	(junction
-		(at 26.67 196.85)
+		(at 77.47 177.8)
 		(diameter 0)
 		(color 0 0 0 0)
 	)
 	(junction
-		(at 77.47 177.8)
+		(at 67.31 177.8)
 		(diameter 0)
 		(color 0 0 0 0)
 	)
 	(junction
-		(at 67.31 177.8)
+		(at 184.15 170.18)
 		(diameter 0)
 		(color 0 0 0 0)
@@
 	)
 	(junction
+		(at 184.15 177.8)
+		(diameter 0)
+		(color 0 0 0 0)
+	)
+	(junction
 		(at 74.93 105.41)
 		(diameter 0)
@@
 	)
 	(junction
-		(at 184.15 177.8)
+		(at 106.68 177.8)
 		(diameter 0)
 		(color 0 0 0 0)
 	)
 	(junction
-		(at 106.68 177.8)
+		(at 194.31 170.18)
 		(diameter 0)
 		(color 0 0 0 0)
 	)
 	(junction
-		(at 148.59 170.18)
+		(at 158.75 170.18)
 		(diameter 0)
 		(color 0 0 0 0)
@@
 	)
 	(junction
-		(at 148.59 177.8)
+		(at 148.59 170.18)
 		(diameter 0)
 		(color 0 0 0 0)
@@
 	)
 	(junction
+		(at 194.31 177.8)
+		(diameter 0)
+		(color 0 0 0 0)
+	)
+	(junction
 		(at 86.36 196.85)
 		(diameter 0)
@@
 	)
 	(junction
-		(at 194.31 177.8)
-		(diameter 0)
-		(color 0 0 0 0)
-	)
-	(junction
 		(at 292.1 135.89)
 		(diameter 0)
@@
 	(wire
 		(pts
+			(xy 158.75 177.8) (xy 168.91 177.8)
+		)
+		(stroke
+			(width 0)
+			(type default)
+		)
+	)
+	(wire
+		(pts
 			(xy 199.39 115.57) (xy 204.47 115.57)
 		)
@@
 	(wire
 		(pts
-			(xy 194.31 177.8) (xy 204.47 177.8)
-		)
-		(stroke
-			(width 0)
-			(type default)
-		)
-	)
-	(wire
-		(pts
 			(xy 86.36 196.85) (xy 96.52 196.85)
 		)
@@
 	(wire
 		(pts
-			(xy 158.75 177.8) (xy 168.91 177.8)
-		)
-		(stroke
-			(width 0)
-			(type default)
-		)
-	)
-	(wire
-		(pts
 			(xy 148.59 167.64) (xy 148.59 170.18)
 		)
@@
 	(wire
 		(pts
-			(xy 158.75 170.18) (xy 168.91 170.18)
+			(xy 397.51 110.49) (xy 396.24 110.49)
 		)
 		(stroke
@@
 	(wire
 		(pts
-			(xy 397.51 110.49) (xy 396.24 110.49)
+			(xy 158.75 170.18) (xy 168.91 170.18)
 		)
 		(stroke
@@
 	(wire
 		(pts
-			(xy 194.31 170.18) (xy 204.47 170.18)
-		)
-		(stroke
-			(width 0)
-			(type default)
-		)
-	)
-	(wire
-		(pts
 			(xy 203.2 189.23) (xy 203.2 193.04)
 		)
@@
 	(wire
 		(pts
+			(xy 194.31 170.18) (xy 204.47 170.18)
+		)
+		(stroke
+			(width 0)
+			(type default)
+		)
+	)
+	(wire
+		(pts
 			(xy 86.36 189.23) (xy 96.52 189.23)
 		)
@@
 	(wire
 		(pts
+			(xy 194.31 177.8) (xy 204.47 177.8)
+		)
+		(stroke
+			(width 0)
+			(type default)
+		)
+	)
+	(wire
+		(pts
 			(xy 238.76 168.91) (xy 240.03 168.91)
 		)
@@
 		)
 	)
-	(global_label "AEN"
+	(global_label "BALE"
 		(shape input)
 		(at 360.68 144.78 180)
@@
 		)
 		(property "Intersheetrefs" "${INTERSHEET_REFS}"
-			(at 354.1267 144.78 0)
+			(at 353.1591 144.78 0)
 			(effects
 				(font
@@
 		)
 	)
-	(global_label "BALE"
+	(global_label "GND"
 		(shape input)
-		(at 360.68 147.32 180)
+		(at 148.59 180.34 0)
 		(fields_autoplaced yes)
 		(effects
@@
 				(size 1.27 1.27)
 			)
-			(justify right)
+			(justify left)
 		)
 		(property "Intersheetrefs" "${INTERSHEET_REFS}"
-			(at 353.1591 147.32 0)
+			(at 155.4457 180.34 0)
 			(effects
 				(font
 					(size 1.27 1.27)
 				)
-				(justify right)
+				(justify left)
 				(hide yes)
 			)
 		)
 	)
-	(global_label "GND"
+	(global_label "SERIRQ"
 		(shape input)
-		(at 148.59 180.34 0)
+		(at 281.94 175.26 180)
 		(fields_autoplaced yes)
 		(effects
@@
 				(size 1.27 1.27)
 			)
-			(justify left)
+			(justify right)
 		)
 		(property "Intersheetrefs" "${INTERSHEET_REFS}"
-			(at 155.4457 180.34 0)
+			(at 272.121 175.26 0)
 			(effects
 				(font
 					(size 1.27 1.27)
 				)
-				(justify left)
+				(justify right)
 				(hide yes)
 			)
 		)
 	)
-	(global_label "SERIRQ"
+	(global_label "AEN"
 		(shape input)
-		(at 281.94 175.26 180)
+		(at 360.68 147.32 180)
 		(fields_autoplaced yes)
 		(effects
@@
 		)
 		(property "Intersheetrefs" "${INTERSHEET_REFS}"
-			(at 272.121 175.26 0)
+			(at 354.1267 147.32 0)
 			(effects
 				(font
@@
 	(symbol
 		(lib_id "Device:C_US")
-		(at 194.31 173.99 0)
+		(at 194.31 173.99 180)
 		(unit 1)
 		(exclude_from_sim no)
@@
 		(dnp no)
 		(property "Reference" "C32"
-			(at 196.596 172.974 0)
+			(at 192.024 175.006 0)
 			(effects
 				(font
@@
 		)
 		(property "Value" "100nF"
-			(at 196.596 175.26 0)
+			(at 192.024 172.72 0)
 			(effects
 				(font
@@
 	(symbol
 		(lib_id "Device:C_US")
-		(at 204.47 173.99 0)
+		(at 204.47 173.99 180)
 		(unit 1)
 		(exclude_from_sim no)
@@
 		(dnp no)
 		(property "Reference" "C33"
-			(at 206.756 172.974 0)
+			(at 202.184 175.006 0)
 			(effects
 				(font
@@
 		)
 		(property "Value" "100uF"
-			(at 206.756 175.514 0)
+			(at 202.184 172.466 0)
 			(effects
 				(font
@@
 	(symbol
 		(lib_id "Device:C_US")
-		(at 184.15 173.99 0)
+		(at 184.15 173.99 180)
 		(unit 1)
 		(exclude_from_sim no)
@@
 		(dnp no)
 		(property "Reference" "C19"
-			(at 186.436 172.974 0)
+			(at 181.864 175.006 0)
 			(effects
 				(font
@@
 		)
 		(property "Value" "100nF"
-			(at 186.436 175.514 0)
+			(at 181.864 172.466 0)
 			(effects
 				(font
@@
 	(symbol
 		(lib_id "Device:C_US")
-		(at 168.91 173.99 0)
+		(at 168.91 173.99 180)
 		(unit 1)
 		(exclude_from_sim no)
@@
 		(dnp no)
 		(property "Reference" "C18"
-			(at 171.196 172.974 0)
+			(at 166.624 175.006 0)
 			(effects
 				(font
@@
 		)
 		(property "Value" "47uF"
-			(at 171.196 175.514 0)
+			(at 166.624 172.466 0)
 			(effects
 				(font
@@
 	(symbol
 		(lib_id "Device:C_US")
-		(at 148.59 173.99 0)
+		(at 148.59 173.99 180)
 		(unit 1)
 		(exclude_from_sim no)
@@
 		(dnp no)
 		(property "Reference" "C16"
-			(at 150.876 172.974 0)
+			(at 146.304 175.006 0)
 			(effects
 				(font
@@
 		)
 		(property "Value" "100nF"
-			(at 150.876 175.514 0)
+			(at 146.304 172.466 0)
 			(effects
 				(font
@@
 	(symbol
 		(lib_id "Device:C_US")
-		(at 158.75 173.99 0)
+		(at 158.75 173.99 180)
 		(unit 1)
 		(exclude_from_sim no)
@@
 		(dnp no)
 		(property "Reference" "C17"
-			(at 161.036 172.974 0)
+			(at 156.464 175.006 0)
 			(effects
 				(font
@@
 		)
 		(property "Value" "100nF"
-			(at 161.036 175.26 0)
+			(at 156.464 172.72 0)
 			(effects
 				(font

Commit message: Errata 1 and DRQ Pull Down Fix
Parts:
- RN1: value R_Net_10_10k -> R_Net_10_4k7
Changed lines of the file:
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@@
 			)
 		)
-		(property "Value" "R_Net_10_10k"
+		(property "Value" "R_Net_10_4k7"
 			(at 244.856 99.06 90)
 			(effects
