File: ProtoPCI/ProtoPCI.kicad_pcb (KiCad board)
At the start: 2 copper layers, 101.2 x 50.3 mm, 7 parts, among them J1 Bus_PCI_32bit_Universal, J2 Conn_01x11_Pin, J3 Conn_01x11_Pin, J4 Conn_01x11_Pin, J5 Conn_01x11_Pin, J6 Conn_01x36_Pin, J7 Conn_01x36_Pin

Commit message: PCI Breakout Proto
Parts:
- added G***: LOGO, DFT:DFT_SS_Small, B.Cu at (157.7, 91.6)
- added G***: LOGO, DFT:DFT_Logo_Small, B.Cu at (188.9, 91.6)
- moved J3 11.1 mm to (116.0, 106.0)
- moved J2 11.0 mm to (141.4, 100.9)
- moved J5 11.0 mm to (179.5, 106.0)
- moved J4 11.0 mm to (204.9, 100.9)
- moved J7 0.30 mm to (116.0, 80.6)
- moved J6 0.28 mm to (204.9, 75.5)
Routing:
- net Net-(J2-Pin_4): track 38.5 -> 20.4 mm, vias 1 -> 0
- net Net-(J2-Pin_1): track 39.9 -> 23.0 mm, vias 1 -> 0
- net Net-(J7-Pin_33): track 64.0 -> 47.9 mm, vias 1 -> 0
- net Net-(J1-AD[08]): track 31.2 -> 15.3 mm, vias 2 -> 0
- net Net-(J1-AD[07]): track 30.5 -> 14.7 mm, vias 3 -> 0
- net Net-(J1--12V): track 27.7 -> 14.7 mm, vias 1 -> 0
- net Net-(J1-TDI): track 30.4 -> 18.2 mm
- net Net-(J1-~{INTA#}): track 31.3 -> 19.3 mm, vias 1 -> 0
- net Net-(J3-Pin_3): track 25.3 -> 13.7 mm, vias 1 -> 0
- net Net-(J1-TDO): track 24.8 -> 13.1 mm, vias 1 -> 0
- net Net-(J1-TCK): track 25.8 -> 14.2 mm, vias 1 -> 0
- net Net-(J3-Pin_5): track 24.3 -> 12.7 mm, vias 1 -> 0
- net Net-(J1-TMS): track 30.3 -> 18.8 mm, vias 1 -> 0
- net Net-(J1-~{TRST#}): track 31.4 -> 19.8 mm
- net Net-(J1-+12V): track 30.8 -> 19.3 mm
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Other:
- board text added: "A SIDE"
- board text added: "B SIDE"
- board text added: "PCI Breakout DFT - (DartFrogTek)"

Commit message: Proto PCI Slot/Edge Rev0
Parts:
- added G***: LOGO, DFT:DFT_SS_Small, B.Cu at (146.5, 57.7)
- added G***: LOGO, DFT:DFT_Logo_Small, B.Cu at (177.7, 57.7)
- added J1: Bus_PCI_32bit_Universal_Slot, PCI_Slot:51451541, F.Cu at (110.9, 63.2)
- added J10: Conn_01x11_Pin, Connector_PinHeader_2.54mm:PinHeader_1x11_P2.54mm_Vertical, F.Cu at (168.3, 46.7)
- added J12: Conn_01x11_Pin, Connector_PinHeader_2.54mm:PinHeader_1x11_P2.54mm_Vertical, F.Cu at (130.2, 77.1)
- added J13: Conn_01x36_Pin, Connector_PinHeader_2.54mm:PinHeader_1x36_P2.54mm_Vertical, F.Cu at (193.7, 84.8)
- added J14: Conn_01x11_Pin, Connector_PinHeader_2.54mm:PinHeader_1x11_P2.54mm_Vertical, F.Cu at (193.7, 77.2)
- added J8: Conn_01x11_Pin, Connector_PinHeader_2.54mm:PinHeader_1x11_P2.54mm_Vertical, F.Cu at (104.8, 46.7)
- added J9: Conn_01x36_Pin, Connector_PinHeader_2.54mm:PinHeader_1x36_P2.54mm_Vertical, F.Cu at (104.8, 39.1)
- moved J2 23.2 mm to (130.3, 121.2)
- moved J4 23.2 mm to (193.8, 121.2)
- moved J5 23.2 mm to (168.4, 126.3)
- moved J3 23.2 mm to (104.9, 126.3)
- moved J7 23.2 mm to (104.9, 100.9)
- moved J1 23.2 mm to (148.7, 137.6)
- moved J6 23.2 mm to (193.8, 95.8)
- moved G*** 23.2 mm to (146.6, 111.9)
- moved G*** 23.2 mm to (177.8, 111.9)
Routing:
- net Net-(J1-AD[09]): track 60.3 -> 94.9 mm
- net Net-(J7-Pin_1): track 56.1 -> 89.5 mm
- net Net-(J1-~{RST#}): track 61.2 -> 94.2 mm
- net Net-(J1-AD[10]): track 52.7 -> 85.1 mm
- net Net-(J1-CLK): track 51.3 -> 83.3 mm
- net Net-(J1-AD[11]): track 55.6 -> 87.0 mm
- net Net-(J1-3.3VAUX): track 63.6 -> 94.9 mm
- net Net-(J1-M66EN): track 55.1 -> 85.9 mm
- net Net-(J1-~{GNT#}): track 56.1 -> 86.6 mm
- net Net-(J7-Pin_2): track 53.7 -> 83.8 mm
- net Net-(J6-Pin_2): track 58.0 -> 88.0 mm
- net Net-(J7-Pin_33): track 47.9 -> 77.7 mm
- net Net-(J1-~{REQ#}): track 46.8 -> 76.3 mm
- net Net-(J1-PME#): track 51.7 -> 81.1 mm
- net Net-(J6-Pin_34): track 58.4 -> 87.6 mm
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Other:
- board size 101.2 x 50.3 mm -> 101.2 x 105.6 mm
- board text added: "PCI Slot Breakout DFT - (DartFrogTek)"
