File: ProtoPCI/ProtoPCISlot.kicad_sch (KiCad schematic)
At the start: 14 parts, among them J1 Bus_PCI_32bit_Universal, J10 Conn_01x11_Pin, J11 Bus_PCI_32bit_Universal_Slot, J12 Conn_01x11_Pin, J13 Conn_01x36_Pin, J14 Conn_01x11_Pin, J2 Conn_01x11_Pin, J3 Conn_01x11_Pin, J4 Conn_01x11_Pin, J5 Conn_01x11_Pin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

Commit message: Proto PCI Slot/Edge Rev0
Parts:
- removed J10, J12, J14, J8: Conn_01x11_Pin, Connector_PinHeader_2.54mm:PinHeader_1x11_P2.54mm_Vertical, symbol Connector:Conn_01x11_Pin
- removed J11: Bus_PCI_32bit_Universal_Slot, PCI_Slot:51451541, symbol Connector:Bus_PCI_32bit_Universal
- removed J13, J9: Conn_01x36_Pin, Connector_PinHeader_2.54mm:PinHeader_1x36_P2.54mm_Vertical, symbol Connector:Conn_01x36_Pin
- J1: value Bus_PCI_32bit_Universal -> Bus_PCI_32bit_Universal_Slot; footprint Connector_PCBEdge:BUS_PCI -> PCI_Slot:51451541
Other:
- moved on the sheet: J2, J3, J4, J5, J6, J7
